Commit message: spawning 2 robots but time jumping problem (need correction)

File: src/pearlguard_description/pguard.xacro (robot description, xacro)
@@ -12,12 +12,12 @@
   <xacro:include filename="urdf/materials.xacro" />
   <xacro:include filename="urdf/inertia.xacro" />
-  <link name="base_footprint" />
+  <link name="$(arg namespace)/base_footprint" />
   <joint name="base_joint" type="fixed">
-    <parent link="base_footprint"/>
-    <child link="base_link"/>
+    <parent link="$(arg namespace)/base_footprint"/>
+    <child link="$(arg namespace)/base_link"/>
     <origin xyz="0 0 0.20" rpy="0 0 0" />
   </joint>
   <!-- base_link -->
-  <link name='base_link'>
+  <link name='$(arg namespace)/base_link'>
     <visual>
       <origin xyz="0.0 0.0 0" rpy="0 0 0"/>
@@ -48,14 +48,14 @@
   <!-- Dome -->
   <xacro:include filename="urdf/dome.urdf.xacro" />
-  <xacro:dome xyz="0 0 0.65" parent="base_link"/>
+  <xacro:dome xyz="0 0 0.65" parent="$(arg namespace)/base_link"/>
   <!-- Wheels -->
   <xacro:include filename="urdf/wheel.urdf.xacro" />
-  <xacro:wheel name="frontLeft"  xyz="${+Lxf} ${+Lw/2} ${-Lz}" parent="base_link"/>
-  <xacro:wheel name="rearLeft"   xyz="${-Lxr} ${+Lw/2} ${-Lz}" parent="base_link"/>
-  <xacro:wheel name="frontRight" xyz="${+Lxf} ${-Lw/2} ${-Lz}" parent="base_link"/>
-  <xacro:wheel name="rearRight"  xyz="${-Lxr} ${-Lw/2} ${-Lz}" parent="base_link"/>
+  <xacro:wheel name="frontLeft"  xyz="${+Lxf} ${+Lw/2} ${-Lz}" parent="$(arg namespace)/base_link"/>
+  <xacro:wheel name="rearLeft"   xyz="${-Lxr} ${+Lw/2} ${-Lz}" parent="$(arg namespace)/base_link"/>
+  <xacro:wheel name="frontRight" xyz="${+Lxf} ${-Lw/2} ${-Lz}" parent="$(arg namespace)/base_link"/>
+  <xacro:wheel name="rearRight"  xyz="${-Lxr} ${-Lw/2} ${-Lz}" parent="$(arg namespace)/base_link"/>
   <!-- Lidar -->
   <xacro:include filename="urdf/VLP-16.urdf.xacro"/>
-  <xacro:VLP-16 parent="base_link" name="velodyne" topic="ouster/points" hz="10" samples="360" gpu="true" min_range="0.45" >
+  <xacro:VLP-16 parent="$(arg namespace)/base_link" name="velodyne" topic="ouster/points" hz="10" samples="360" gpu="true" min_range="0.45" >
     <origin xyz="0.50 0.00 0.65" rpy="0 0 0" />
   </xacro:VLP-16>
@@ -63,4 +63,4 @@
   <xacro:include filename="urdf/imu.urdf.xacro"/>
   <xacro:property name="M_PI" value="3.1415926535897931" />
-  <xacro:sensor_imu parent="base_link" name="imu" colour="blue" imu_px="0.192" imu_py="0.0" imu_pz="${0.01}" imu_or="0.0" imu_op="${-M_PI/2.0}" imu_oy="0.0"/>
+  <xacro:sensor_imu parent="$(arg namespace)/base_link" name="imu" colour="blue" imu_px="0.192" imu_py="0.0" imu_pz="${0.01}" imu_or="0.0" imu_op="${-M_PI/2.0}" imu_oy="0.0"/>
 </robot>

File: src/pearlguard_description/urdf/VLP-16.urdf.xacro (robot description, xacro)
@@ -6,7 +6,7 @@
       <xacro:insert_block name="origin" />
       <parent link="${parent}"/>
-      <child link="${name}_base_link"/>
+      <child link="$(arg namespace)/${name}_base_link"/>
     </joint>
-    <link name="${name}_base_link">
+    <link name="$(arg namespace)/${name}_base_link">
       <inertial>
         <mass value="0.83"/>
@@ -35,8 +35,8 @@
     <joint name="${name}_base_scan_joint" type="fixed" >
       <origin xyz="0 0 0.0377" rpy="0 0 0" />
-      <parent link="${name}_base_link" />
-      <child link="${name}"/>
+      <parent link="$(arg namespace)/${name}_base_link" />
+      <child link="$(arg namespace)/${name}"/>
     </joint>
-    <link name="${name}">
+    <link name="$(arg namespace)/${name}">
       <inertial>
         <mass value="0.01"/>
@@ -52,5 +52,5 @@
     </link>
     <!-- Gazebo requires the velodyne_gazebo_plugins package -->
-    <gazebo reference="${name}">
+    <gazebo reference="$(arg namespace)/${name}">
   <sensor name="${name}_lidar" type="gpu_lidar">
     <always_on>true</always_on>
@@ -58,5 +58,5 @@
     <update_rate>${hz}</update_rate>
     <topic>$(arg namespace)/${topic}</topic>
-    <gz_frame_id>${name}</gz_frame_id>
+    <gz_frame_id>$(arg namespace)/${name}</gz_frame_id>
     <lidar>
       <scan>

File: src/pearlguard_description/urdf/dome.urdf.xacro (robot description, xacro)
@@ -5,5 +5,5 @@
   <xacro:property name="domeMass" value="10"/>
   <xacro:macro name="dome" params="xyz parent">
-    <link name="dome">
+    <link name="$(arg namespace)/dome">
       <visual>
         <origin xyz="0 0 0" rpy="0 0 ${PI/2}" />
@@ -21,5 +21,5 @@
     <joint name="dome_joint" type="continuous">
         <parent link="${parent}"/>
-        <child link="dome"/>
+        <child link="$(arg namespace)/dome"/>
         <origin xyz="${xyz}" rpy="0 0 0" />
         <axis xyz="0 0 1" />
@@ -27,5 +27,5 @@
         <joint_properties damping="0.0" friction="0.0"/>
     </joint>
-    <gazebo reference="dome">
+    <gazebo reference="$(arg namespace)/dome">
       <mu1 value=".62"/>
       <mu2 value=".62"/>

File: src/pearlguard_description/urdf/imu.urdf.xacro (robot description, xacro)
@@ -3,5 +3,5 @@
   <xacro:include filename="imusensor_gazebo.urdf.xacro"/>
   <xacro:macro name="sensor_imu" params="parent name colour imu_px imu_py imu_pz imu_or imu_op imu_oy">
-    <link name="${name}_link">
+    <link name="$(arg namespace)/${name}_link">
       <inertial>
         <mass value="0.01"/>
@@ -19,8 +19,8 @@
     <joint name="${name}_joint" type="fixed">
       <parent link="${parent}"/>
-      <child link="${name}_link"/>
+      <child link="$(arg namespace)/${name}_link"/>
       <origin xyz="${imu_px} ${imu_py} ${imu_pz}" rpy="${imu_or} ${imu_op} ${imu_oy}"/>
     </joint>
-    <gazebo reference="${name}_link">
+    <gazebo reference="$(arg namespace)/${name}_link">
       <material>Gazebo/blue</material>
     </gazebo>

File: src/pearlguard_description/urdf/pguard_x.gazebo.xacro (robot description, xacro)
@@ -2,23 +2,23 @@
 <robot xmlns:xacro="http://www.ros.org/wiki/xacro">
 <xacro:arg name="namespace" default=""/>
-<gazebo reference="base_link">
-<material>Gazebo/Orange</material>
+<gazebo reference="$(arg namespace)/base_link">
+  <material>Gazebo/Orange</material>
 </gazebo>
 <!-- 4WD differential drive (replaces Classic skid_steer + ros_control) -->
 <!-- 4WD differential drive (replaces Classic skid_steer + ros_control) -->
 <gazebo>
-<plugin filename="libgz-sim-diff-drive-system.so" name="gz::sim::systems::DiffDrive">
-<left_joint>frontLeft_wheel_joint</left_joint>
-<left_joint>rearLeft_wheel_joint</left_joint>
-<right_joint>frontRight_wheel_joint</right_joint>
-<right_joint>rearRight_wheel_joint</right_joint>
-<wheel_separation>0.920</wheel_separation>
-<wheel_radius>0.200</wheel_radius>
-<topic>$(arg namespace)/cmd_vel</topic>
-<odom_topic>$(arg namespace)/odom</odom_topic>
-<frame_id>odom</frame_id>
-<child_frame_id>base_footprint</child_frame_id>
-<publish_odom_tf>false</publish_odom_tf>
-</plugin>
+  <plugin filename="libgz-sim-diff-drive-system.so" name="gz::sim::systems::DiffDrive">
+    <left_joint>$(arg namespace)/frontLeft_wheel_joint</left_joint>
+    <left_joint>$(arg namespace)/rearLeft_wheel_joint</left_joint>
+    <right_joint>$(arg namespace)/frontRight_wheel_joint</right_joint>
+    <right_joint>$(arg namespace)/rearRight_wheel_joint</right_joint>
+    <wheel_separation>0.920</wheel_separation>
+    <wheel_radius>0.200</wheel_radius>
+    <topic>$(arg namespace)/cmd_vel</topic>
+    <odom_topic>$(arg namespace)/odom</odom_topic>
+    <frame_id>odom</frame_id>
+    <child_frame_id>$(arg namespace)/base_footprint</child_frame_id>
+    <publish_odom_tf>false</publish_odom_tf>
+  </plugin>
 </gazebo>
 <!-- Publish joint states for ros2_control / ros2 topic bridge -->
@@ -29,16 +29,16 @@
 </gazebo>
 <!-- GPS / NavSat (replaces Classic hector_gazebo_ros_gps) -->
-<gazebo reference="base_link">
-<sensor name="navsat_sensor" type="navsat">
-<always_on>1</always_on>
-<update_rate>10</update_rate>
-<visualize>true</visualize>
-<gz_frame_id>base_footprint</gz_frame_id>
-<topic>$(arg namespace)/navsat</topic>
-<plugin filename="libgz-sim-navsat-system.so" name="gz::sim::systems::NavSat">
-<reference_latitude>35.8173</reference_latitude>
-<reference_longitude>10.5912</reference_longitude>
-</plugin>
-</sensor>
+<gazebo reference="$(arg namespace)/base_link">
+  <sensor name="navsat_sensor" type="navsat">
+    <always_on>1</always_on>
+    <update_rate>10</update_rate>
+    <visualize>true</visualize>
+    <gz_frame_id>$(arg namespace)/base_footprint</gz_frame_id>
+    <topic>$(arg namespace)/navsat</topic>
+    <plugin filename="libgz-sim-navsat-system.so" name="gz::sim::systems::NavSat">
+      <reference_latitude>35.8173</reference_latitude>
+      <reference_longitude>10.5912</reference_longitude>
+    </plugin>
+  </sensor>
 </gazebo>
 </robot>

File: src/pearlguard_description/urdf/wheel.urdf.xacro (robot description, xacro)
@@ -4,5 +4,5 @@
   <xacro:property name="wheelMass" value="5"/>
   <xacro:macro name="wheel" params="name xyz parent">
-    <link name="${name}_wheel">
+    <link name="$(arg namespace)/${name}_wheel">
       <collision>
         <origin xyz="0 0 0" rpy="0 ${PI/2} ${PI/2}" />
@@ -24,7 +24,7 @@
       </inertial>
     </link>
-    <joint name="${name}_wheel_joint" type="continuous">
+    <joint name="$(arg namespace)/${name}_wheel_joint" type="continuous">
         <parent link="${parent}"/>
-        <child link="${name}_wheel"/>
+        <child link="$(arg namespace)/${name}_wheel"/>
         <origin xyz="${xyz}" rpy="0 0 0" />
         <axis xyz="0 1 0" />
@@ -32,5 +32,5 @@
         <joint_properties damping="0.0" friction="0.0"/>
     </joint>
-    <gazebo reference="${name}_wheel">
+    <gazebo reference="$(arg namespace)/${name}_wheel">
       <mu1 value="1.2"/>
       <mu2 value="1.0"/>
