Commit message: add another robot, change robots color , fix the rsobridge connection failure

File: src/pearlguard_description/urdf/materials.xacro (robot description, xacro)
@@ -3,4 +3,7 @@
   <material name="black">
     <color rgba="0.0 0.0 0.0 1.0"/>
+  </material>
+  <material name="dark_grey">
+    <color rgba="0.15 0.15 0.15 1.0"/>
   </material>
   <material name="blue">

File: src/pearlguard_description/urdf/pguard_x.gazebo.xacro (robot description, xacro)
@@ -3,5 +3,11 @@
 <xacro:arg name="namespace" default=""/>
 <gazebo reference="$(arg namespace)/base_link">
-  <material>Gazebo/Orange</material>
+  <visual>
+    <material>
+      <ambient>0.25 0.25 0.25 1</ambient>
+      <diffuse>0.25 0.25 0.25 1</diffuse>
+      <specular>0.2 0.2 0.2 1</specular>
+    </material>
+  </visual>
 </gazebo>
 <!-- 4WD differential drive (replaces Classic skid_steer + ros_control) -->
